File: KiCAD files/BARBIE_PCB/BARBIE_PCB.kicad_sch (KiCad schematic)
At the start: 0 parts

Commit message: Added a voltage regulators and a switch. Still need to finish adding footprints.
Parts:
- added BT1: Battery_Cell, symbol Device:Battery_Cell
- added C1, C11: 100nF, Inductor_SMD:L_0402_1005Metric, symbol Device:C_Small
- added C10, C12, C2, C3, C4, C6, C8, C9: 10uF, Capacitor_SMD:C_0603_1608Metric_Pad1.08x0.95mm_HandSolder, symbol Device:C_Small
- added C13, C14, C15, C16, C17, C5: 22uF, Inductor_SMD:L_0805_2012Metric, symbol Device:C_Small
- added C7: C, symbol Device:C
- added L1, L2: 1.5uH, Inductor_SMD:L_Coilcraft_XxL4020, symbol Device:L_Small
- added Q1, Q2: NMOS, symbol Simulation_SPICE:NMOS
- added R1, R8: 470k, Resistor_SMD:R_0805_2012Metric, symbol Device:R_Small_US
- added R10, R3: 100k, symbol Device:R_Small_US
- added R11, R4, R5: 10k, Resistor_SMD:R_1206_3216Metric, symbol Device:R_Small_US
- added R12: 220k, Resistor_SMD:R_0805_2012Metric, symbol Device:R_Small_US
- added R2: 150k, Resistor_SMD:R_0805_2012Metric, symbol Device:R_Small_US
- added R6: 1M, symbol Device:R_Small_US
- added R7: R_Small_US, symbol Device:R_Small_US
- added R9: 120k, Resistor_SMD:R_0603_1608Metric, symbol Device:R_Small_US
- added SW1: SW_SPDT, symbol Switch:SW_SPDT
- added U1, U2: TPS60701RNMR, Package_SO:MSOP-10_3x3mm_P0.5mm, symbol Our_Library:TPS60701RNMR
- added U3: TPS3831, Package_SON:Texas_X2SON-4_1x1mm_P0.65mm, symbol Power_Supervisor:TPS3831
Connections:
- new net: C11.1, U2.3 (VAUX)
- new net: R4.2, U1.1 (PS/SYNC), U1.14 (EN)
- new net: L1.2, U1.11 (L1)
- new net: R3.2, U1.2 (PG)
- new net: C1.1, U1.3 (VAUX)
- new net: R1.2, R2.1, U1.5 (FB)
- new net: L1.1, U1.9 (L2)
- new net: C7.1, R6.2
- new net: R7.2, SW1.3 (C)
- new net: Q1.2 (G), R6.1, SW1.2 (B)
- new net: R5.2, U2.1 (PS/SYNC), U2.14 (EN)
- new net: L2.2, U2.11 (L1)
- new net: R10.2, U2.2 (PG)
- new net: R12.2, R9.1, U2.5 (FB)
- new net: L2.1, U2.9 (L2)
- new net: R12.1, R8.2
- new net: R11.1, R9.2
- new net 3V3: C16.1, C17.1, C4.1, C5.1, R1.1, R3.1, U1.7 (VOUT), U1.8 (VOUT)
- new net 5V: C12.1, C13.1, C14.1, C15.1, R10.1, R8.1, U2.7 (VOUT), U2.8 (VOUT)
- new net BATTERY_OK: Q2.2 (G), U3.1 (~{RESET})
- new net GND: BT1.2 (-), C7.2, Q1.3 (S), Q2.3 (S), R7.1, U3.3 (GND)
- new net GNDREF: C1.2, C10.2, C11.2, C12.2, C13.2, C14.2, C15.2, C16.2, C17.2, C2.2, C3.2, C4.2, C5.2, C6.2, C8.2, C9.2, Q1.1 (D), Q2.1 (D), R11.2, R2.2, U1.10 (PGND), U1.4 (GND), U1.6 (FB2), U2.10 (PGND), U2.4 (GND), U2.6 (FB2)
- new net V_BATTERY: BT1.1 (+), C10.1, C2.1, C3.1, C6.1, C8.1, C9.1, R4.1, R5.1, SW1.1 (A), U1.12 (VIN), U1.13 (VIN), U2.12 (VIN), U2.13 (VIN), U3.4 (VDD)
Other:
- note added: "3V3 and 5V voltage regulation circuits. Capacitor and resistor values haven't been chosen yet."
- note added: "3V3 voltage regulator"
- note added: "5V voltage regulator"
- note added: "Device can operate in power save mode if PS/SYNC is set to high."
- note added: "Disables power to the sensor module when the battery is critically low."
- note added: "Supervisor IC to monitor battery health"
- note added: "Switch circuit"
- note added: "This is Hannah's spot"

Commit message: Starting PCB layout and tracing
Parts:
- added C_ESP32: C_Polarized_US, Capacitor_THT:CP_Radial_D6.3mm_P2.50mm, symbol Device:C_Polarized_US
- added JP_ESP32_2, JP_ESP32_9: SolderJumper_2_Open, Jumper:SolderJumper-2_P1.3mm_Open_RoundedPad1.0x1.5mm, symbol Jumper:SolderJumper_2_Open
- added J_Config1: Conn_02x03_Odd_Even, Connector_PinSocket_2.54mm:PinSocket_2x03_P2.54mm_Vertical, symbol Connector_Generic:Conn_02x03_Odd_Even
- added J_Mounting1, J_Receive1: Conn_01x06_Pin, Connector_PinSocket_2.54mm:PinSocket_1x06_P2.54mm_Vertical, symbol Connector:Conn_01x06_Pin
- added J_Program1: Conn_01x04_Socket, Connector_PinSocket_2.54mm:PinSocket_1x04_P2.54mm_Vertical, symbol Connector:Conn_01x04_Socket
- added J_Provide1, J_Provide2: Conn_01x13, Connector_PinSocket_2.54mm:PinSocket_1x13_P2.54mm_Vertical, symbol Connector_Generic:Conn_01x13
- added J_SD_Card1: Micro_SD_Card, Connector_Card:microSD_HC_Molex_47219-2001, symbol Connector:Micro_SD_Card
- added J_Share1: Conn_01x02_Pin, Connector_PinHeader_2.54mm:PinHeader_1x02_P2.54mm_Vertical, symbol Connector:Conn_01x02_Pin
- added J_USB_C1: USB_C_Receptacle_USB2.0_16P, Connector_USB:USB_C_Receptacle_GCT_USB4105-xx-A_16P_TopMnt_Horizontal, symbol Connector:USB_C_Receptacle_USB2.0_16P
- added R_CC1, R_CC2: 5.6kR, Resistor_SMD:R_0805_2012Metric, symbol Device:R_Small_US
- added R_D+1, R_D-1: 22R, Resistor_SMD:R_0402_1005Metric, symbol Device:R_Small_US
- added R_ESP32_3, R_ESP32_4, R_ESP32_46, R_MISO1, R_MOSI1, R_SCL1, R_SDA1, R_SD_CARD1, R_SD_CARD2, R_SD_CARD_CS1, R_nReset1: 1MR, Resistor_SMD:R_0402_1005Metric, symbol Device:R_Small_US
- added SW_nReset1: SW_Push, Button_Switch_THT:SW_PUSH_6mm, symbol Switch:SW_Push
- added U_ESP32: ESP32-S3-WROOM-1, RF_Module:ESP32-S3-WROOM-1U, symbol RF_Module:ESP32-S3-WROOM-1
Connections:
- net GNDREF: now also C_ESP32.2, JP_ESP32_2.1 (A), JP_ESP32_9.1 (A), J_Config1.2 (Pin_2), J_Config1.4 (Pin_4), J_Config1.6 (Pin_6), J_Program1.1 (Pin_1), J_Provide1.1 (Pin_1), J_Provide2.13 (Pin_13), J_Receive1.1 (Pin_1), J_SD_Card1.6 (VSS), J_Share1.2 (Pin_2), J_USB_C1.A1 (GND), J_USB_C1.A12 (GND), J_USB_C1.B1 (GND), J_USB_C1.B12 (GND), R_CC1.2, R_CC2.2, SW_nReset1.2, U_ESP32.1 (GND), U_ESP32.40 (GND), U_ESP32.41 (GND)
- new net: J_USB_C1.A5 (CC1), R_CC1.1
- new net: J_USB_C1.B5 (CC2), R_CC2.1
- new net: R_D+1.1, U_ESP32.14 (USB_D+)
- new net: R_D-1.1, U_ESP32.13 (USB_D-)
- new net: J_SD_Card1.1 (DAT2), R_SD_CARD2.2
- new net: R_ESP32_3.2, U_ESP32.15 (IO3)
- new net: JP_ESP32_9.2 (B), R_ESP32_46.2, U_ESP32.16 (IO46)
- new net: JP_ESP32_2.2 (B), R_ESP32_4.2, U_ESP32.27 (IO0)
- new net: J_SD_Card1.8 (DAT1), R_SD_CARD1.2
- new net +3V3: C_ESP32.1, J_Provide1.2 (Pin_2), J_Receive1.2 (Pin_2), J_SD_Card1.4 (VDD), R_ESP32_3.1, R_ESP32_4.1, R_ESP32_46.1, R_MISO1.1, R_MOSI1.1, R_SCL1.1, R_SDA1.1, R_SD_CARD1.1, R_SD_CARD2.1, R_SD_CARD_CS1.1, R_nReset1.1, U_ESP32.2 (3V3)
- new net +5V: J_Provide1.3 (Pin_3), J_Receive1.3 (Pin_3)
- new net AD1: J_Provide1.12 (Pin_12), U_ESP32.39 (IO1)
- new net AD2: J_Provide1.13 (Pin_13), U_ESP32.38 (IO2)
- new net AD4: J_Provide2.1 (Pin_1), U_ESP32.4 (IO4)
- new net AD5: J_Provide2.2 (Pin_2), U_ESP32.5 (IO5)
- new net AD6: J_Provide2.3 (Pin_3), U_ESP32.6 (IO6)
- new net AD7: J_Provide2.4 (Pin_4), U_ESP32.7 (IO7)
- new net CS_SD_Card: J_SD_Card1.2 (DAT3/CD), R_SD_CARD_CS1.2, U_ESP32.18 (IO10)
- new net Config1: J_Config1.1 (Pin_1), U_ESP32.34 (IO41)
- new net Config2: J_Config1.3 (Pin_3), U_ESP32.35 (IO42)
- new net Config3: J_Config1.5 (Pin_5), U_ESP32.26 (IO45)
- new net D14: J_Provide2.5 (Pin_5), U_ESP32.22 (IO14)
- new net D15: J_Provide2.6 (Pin_6), U_ESP32.8 (IO15)
- new net D16: J_Provide2.7 (Pin_7), U_ESP32.9 (IO16)
- new net D17: J_Provide2.8 (Pin_8), U_ESP32.10 (IO17)
- new net D18: J_Provide2.9 (Pin_9), U_ESP32.11 (IO18)
- new net D38: J_Provide2.10 (Pin_10), U_ESP32.31 (IO38)
- new net D39: J_Provide2.11 (Pin_11), U_ESP32.32 (IO39)
- new net D40: J_Provide2.12 (Pin_12), U_ESP32.33 (IO40)
- new net I2C_SCL: J_Provide1.8 (Pin_8), J_Receive1.4 (Pin_4), R_SCL1.2, U_ESP32.17 (IO9)
- new net I2C_SDA: J_Provide1.7 (Pin_7), J_Receive1.5 (Pin_5), R_SDA1.2, U_ESP32.12 (IO8)
- new net Low_Battery: J_Receive1.6 (Pin_6), U_ESP32.25 (IO48)
- new net SPI_MISO: J_Provide1.9 (Pin_9), J_SD_Card1.7 (DAT0), R_MISO1.2, U_ESP32.21 (IO13)
- new net SPI_MOSI: J_Provide1.10 (Pin_10), J_SD_Card1.3 (CMD), R_MOSI1.2, U_ESP32.19 (IO11)
- new net SPI_SCK: J_Provide1.11 (Pin_11), J_SD_Card1.5 (CLK), U_ESP32.20 (IO12)
- new net UART_RX: J_Provide1.5 (Pin_5), U_ESP32.37 (TXD0)
- new net UART_TX: J_Provide1.6 (Pin_6), U_ESP32.36 (RXD0)
- new net USB_D+: J_Program1.4 (Pin_4), J_USB_C1.A6 (D+), J_USB_C1.B6 (D+), R_D+1.2
- new net USB_D-: J_Program1.3 (Pin_3), J_USB_C1.A7 (D-), J_USB_C1.B7 (D-), R_D-1.2
- new net USB_V: J_Program1.2 (Pin_2), J_USB_C1.A4 (VBUS), J_USB_C1.A9 (VBUS), J_USB_C1.B4 (VBUS), J_USB_C1.B9 (VBUS)
- new net nEnable_Share: J_Share1.1 (Pin_1), U_ESP32.24 (IO47)
- new net nReset: J_Provide1.4 (Pin_4), R_nReset1.2, SW_nReset1.1, U_ESP32.3 (EN)
- no-connect marks 0 -> 13
