File: KiCAD files/BARBIE_PCB/BARBIE_PCB.kicad_sch (KiCad schematic)
At the start: 0 parts

Commit message: NETWORKS SUBSYSTEM
Complete PCB design of my networks subsystem
Parts:
- added J1: Conn_01x14_Pin, Connector_PinHeader_2.54mm:PinHeader_1x14_P2.54mm_Vertical, symbol Connector:Conn_01x14_Pin
- added J2, J6, J7: Conn_01x12_Pin, Connector_PinHeader_2.54mm:PinHeader_1x12_P2.54mm_Vertical, symbol Connector:Conn_01x12_Pin
- added J3, J5: Conn_01x08_Pin, Connector_PinHeader_2.54mm:PinHeader_1x08_P2.54mm_Vertical, symbol Connector:Conn_01x08_Pin
- added J4: Conn_01x14_Pin, Connector_PinSocket_2.54mm:PinSocket_1x14_P2.54mm_Vertical, symbol Connector:Conn_01x14_Pin
- added U1: ESP32-S3-WROOM-1U-N8, ESP32-WROOM-32UE_N4:ESP32-S3-WROOM-1U_No_holes, symbol ESP32-S3-WROOM-1U.pretty:ESP32-S3-WROOM-1U
- added U2: LORA-CC68-433MHz-TCXO, LORA-CC68-433MHz-TCXO:LORA-CC68-433MHz-TCXO, symbol LORA-CC68-433MHz-TCXO:LoRa-CC68_433MHz-TCXO
- added U3: ATGM332D-5N71, ATGM332D-5NR32:ATGM332D-5NR32, symbol ATGM332D-5NR32:ATGM332D-5NR32
Connections:
- new net: J6.10 (Pin_10), U3.22 (VBAT)
- new net: J6.11 (Pin_11), U3.23 (VCC)
- new net: J6.2 (Pin_2), U3.14 (NC)
- new net: J6.3 (Pin_3), U3.15 (NC)
- new net: J6.4 (Pin_4), U3.16 (TXD2)
- new net: J6.5 (Pin_5), U3.17 (RXD2)
- new net: J6.6 (Pin_6), U3.18 (SDA)
- new net: J6.7 (Pin_7), U3.19 (SCL)
- new net: J6.8 (Pin_8), U3.20 (TXD1)
- new net: J6.9 (Pin_9), U3.21 (RXD1)
- new net: J5.1 (Pin_1), U2.16 (BUSY)
- new net: J5.2 (Pin_2), U2.15 (DIO1)
- new net: J5.3 (Pin_3), U2.14 (NC)
- new net: J5.4 (Pin_4), U2.13 (VCC)
- new net: J5.5 (Pin_5), U2.12 (NC)
- new net: J5.6 (Pin_6), U2.11 (DIO3)
- new net: J5.8 (Pin_8), U2.9 (ANT)
- new net: J3.2 (Pin_2), U2.2 (MISO)
- new net: J3.3 (Pin_3), U2.3 (MOSI)
- new net: J3.4 (Pin_4), U2.4 (SCK)
- new net: J3.5 (Pin_5), U2.5 (NSS)
- new net: J3.6 (Pin_6), U2.6 (NRESET)
- new net: J3.7 (Pin_7), U2.7 (NC)
- new net: J7.12 (Pin_12), U3.1 (NC)
- new net: J7.3 (Pin_3), U3.10 (GND)
- new net: J7.2 (Pin_2), U3.11 (RF_IN)
- new net: J7.11 (Pin_11), U3.2 (Reserved)
- new net: J7.10 (Pin_10), U3.3 (1PPS)
- new net: J7.9 (Pin_9), U3.4 (Reserved)
- new net: J7.8 (Pin_8), U3.5 (NC)
- new net: J7.7 (Pin_7), U3.6 (NC)
- new net: J7.6 (Pin_6), U3.7 (NC)
- new net: J7.5 (Pin_5), U3.8 (nRESET)
- new net: J7.4 (Pin_4), U3.9 (VCC_RF)
- new net 10: J1.10 (Pin_10), U1.10 (IO17)
- new net 11: J1.11 (Pin_11), U1.11 (IO18)
- new net 12: J1.12 (Pin_12), U1.12 (IO8)
- new net 13: J1.13 (Pin_13), U1.13 (IO19)
- new net 14: J1.14 (Pin_14), U1.14 (IO20)
- new net 15: J2.1 (Pin_1), U1.15 (IO3)
- new net 16: J2.2 (Pin_2), U1.16 (IO46)
- new net 17: J2.3 (Pin_3), U1.17 (IO9)
- new net 18: J2.4 (Pin_4), U1.18 (IO10)
- new net 19: J2.5 (Pin_5), U1.19 (IO11)
- new net 2: J1.2 (Pin_2), U1.2 (3V3)
- new net 20: J2.6 (Pin_6), U1.20 (IO12)
- new net 21: J2.7 (Pin_7), U1.21 (IO13)
- new net 22: J2.8 (Pin_8), U1.22 (IO14)
- new net 23: J2.9 (Pin_9), U1.23 (IO21)
- new net 24: J2.10 (Pin_10), U1.24 (IO47)
- new net 25: J2.11 (Pin_11), U1.25 (IO48)
- new net 26: J2.12 (Pin_12), U1.26 (IO45)
- new net 27: J4.1 (Pin_1), U1.27 (IO0)
- new net 28: J4.2 (Pin_2), U1.28 (IO35)
- new net 29: J4.3 (Pin_3), U1.29 (IO36)
- new net 3: J1.3 (Pin_3), U1.3 (EN)
- new net 30: J4.4 (Pin_4), U1.30 (IO37)
- new net 31: J4.5 (Pin_5), U1.31 (IO38)
- new net 32: J4.6 (Pin_6), U1.32 (IO39)
- new net 33: J4.7 (Pin_7), U1.33 (IO40)
- new net 34: J4.8 (Pin_8), U1.34 (IO41)
- new net 35: J4.9 (Pin_9), U1.35 (IO42)
- new net 36: J4.10 (Pin_10), U1.36 (RXD0)
- new net 37: J4.11 (Pin_11), U1.37 (TXD0)
- new net 38: J4.12 (Pin_12), U1.38 (IO2)
- new net 39: J4.13 (Pin_13), U1.39 (IO1)
- new net 4: J1.4 (Pin_4), U1.4 (IO4)
- new net 5: J1.5 (Pin_5), U1.5 (IO5)
- new net 6: J1.6 (Pin_6), U1.6 (IO6)
- new net 7: J1.7 (Pin_7), U1.7 (IO7)
- new net 8: J1.8 (Pin_8), U1.8 (IO15)
- new net 9: J1.9 (Pin_9), U1.9 (IO16)
- new net GND: J1.1 (Pin_1), J3.1 (Pin_1), J3.8 (Pin_8), J4.14 (Pin_14), J5.7 (Pin_7), J6.1 (Pin_1), J6.12 (Pin_12), J7.1 (Pin_1), U1.1 (GND), U1.40 (GND), U1.41 (GND), U2.1 (GND), U2.10 (GND), U2.8 (GND), U3.12 (GND), U3.13 (GND), U3.24 (GND)
Other:
- note added: "NETWORK SUBSYSTEM"

Commit message: Integrated Hannah's schematic into the main schematic
Parts:
- removed J1: Conn_01x14_Pin, Connector_PinHeader_2.54mm:PinHeader_1x14_P2.54mm_Vertical, symbol Connector:Conn_01x14_Pin
- removed J2, J6, J7: Conn_01x12_Pin, Connector_PinHeader_2.54mm:PinHeader_1x12_P2.54mm_Vertical, symbol Connector:Conn_01x12_Pin
- removed J3, J5: Conn_01x08_Pin, Connector_PinHeader_2.54mm:PinHeader_1x08_P2.54mm_Vertical, symbol Connector:Conn_01x08_Pin
- removed J4: Conn_01x14_Pin, Connector_PinSocket_2.54mm:PinSocket_1x14_P2.54mm_Vertical, symbol Connector:Conn_01x14_Pin
- removed U1: ESP32-S3-WROOM-1U-N8, ESP32-WROOM-32UE_N4:ESP32-S3-WROOM-1U_No_holes, symbol ESP32-S3-WROOM-1U.pretty:ESP32-S3-WROOM-1U
- removed U2: LORA-CC68-433MHz-TCXO, LORA-CC68-433MHz-TCXO:LORA-CC68-433MHz-TCXO, symbol LORA-CC68-433MHz-TCXO:LoRa-CC68_433MHz-TCXO
- removed U3: ATGM332D-5N71, ATGM332D-5NR32:ATGM332D-5NR32, symbol ATGM332D-5NR32:ATGM332D-5NR32
- added C1, C11: 100nF, Inductor_SMD:L_0402_1005Metric, symbol Device:C_Small
- added C10, C12, C2, C3, C4, C6, C8, C9: 10uF, Capacitor_SMD:C_0603_1608Metric_Pad1.08x0.95mm_HandSolder, symbol Device:C_Small
- added C13, C14, C15, C16, C17, C5: 22uF, Inductor_SMD:L_0805_2012Metric, symbol Device:C_Small
- added C7: C, symbol Device:C
- added C_ESP32: C_Polarized_US, Capacitor_THT:CP_Radial_D6.3mm_P2.50mm, symbol Device:C_Polarized_US
- added JP1, JP4: SolderJumper_2_Open, symbol Jumper:SolderJumper_2_Open
- added JP3, JP5, JP6, JP_ESP32_2, JP_ESP32_9: SolderJumper_2_Open, Jumper:SolderJumper-2_P1.3mm_Open_RoundedPad1.0x1.5mm, symbol Jumper:SolderJumper_2_Open
- added J_Config1: Conn_02x03_Odd_Even, Connector_PinSocket_2.54mm:PinSocket_2x03_P2.54mm_Vertical, symbol Connector_Generic:Conn_02x03_Odd_Even
- added J_Mounting1, J_Receive1: Conn_01x06_Pin, Connector_PinSocket_2.54mm:PinSocket_1x06_P2.54mm_Vertical, symbol Connector:Conn_01x06_Pin
- added J_Program1: Conn_01x04_Socket, Connector_PinSocket_2.54mm:PinSocket_1x04_P2.54mm_Vertical, symbol Connector:Conn_01x04_Socket
- added J_Provide1, J_Provide2: Conn_01x13, Connector_PinSocket_2.54mm:PinSocket_1x13_P2.54mm_Vertical, symbol Connector_Generic:Conn_01x13
- added J_SD_Card1: Micro_SD_Card, Connector_Card:microSD_HC_Molex_47219-2001, symbol Connector:Micro_SD_Card
- added J_Share1: Conn_01x02_Pin, Connector_PinHeader_2.54mm:PinHeader_1x02_P2.54mm_Vertical, symbol Connector:Conn_01x02_Pin
- added J_USB_C1: USB_C_Receptacle_USB2.0_16P, Connector_USB:USB_C_Receptacle_GCT_USB4105-xx-A_16P_TopMnt_Horizontal, symbol Connector:USB_C_Receptacle_USB2.0_16P
- added L1, L2: 1.5uH, Inductor_SMD:L_Coilcraft_XxL4020, symbol Device:L_Small
- added Q1, Q2: NMOS, symbol Simulation_SPICE:NMOS
- added R1, R8: 470k, Resistor_SMD:R_0805_2012Metric, symbol Device:R_Small_US
- added R10, R3, R6: 100k, symbol Device:R_Small_US
- added R11, R4, R5: 10k, Resistor_SMD:R_1206_3216Metric, symbol Device:R_Small_US
- added R12: 220k, Resistor_SMD:R_0805_2012Metric, symbol Device:R_Small_US
- added R2: 150k, Resistor_SMD:R_0805_2012Metric, symbol Device:R_Small_US
- added R7: R_Small_US, symbol Device:R_Small_US
- added R9: 120k, Resistor_SMD:R_0603_1608Metric, symbol Device:R_Small_US
- added R_CC1, R_CC2: 5.6kR, Resistor_SMD:R_0805_2012Metric, symbol Device:R_Small_US
- added R_D+1, R_D-1: 22R, Resistor_SMD:R_0402_1005Metric, symbol Device:R_Small_US
- added R_ESP32_3, R_ESP32_4, R_ESP32_46, R_MISO1, R_MOSI1, R_SCL1, R_SDA1, R_SD_CARD1, R_SD_CARD2, R_SD_CARD_CS1, R_nReset1: 1MR, Resistor_SMD:R_0402_1005Metric, symbol Device:R_Small_US
- added SW1: SW_SPDT, symbol Switch:SW_SPDT
- added SW2: SW_SPDT, Our_Footprint_Library:SW-TH_1MS1T1B1M1QES-5, symbol Switch:SW_SPDT
- added SW_nReset1: SW_Push, Button_Switch_THT:SW_PUSH_6mm, symbol Switch:SW_Push
- added U1, U2: TPS60701RNMR, Our_Footprint_Library:VQFN-15-HR(3X2.5), symbol Our_Library:TPS60701RNMR
- added U3: TPS3831, Package_SON:Texas_X2SON-4_1x1mm_P0.65mm, symbol Power_Supervisor:TPS3831
- added U_ESP32: ESP32-S3-WROOM-1, RF_Module:ESP32-S3-WROOM-1U, symbol RF_Module:ESP32-S3-WROOM-1
Connections:
- net GND: now also C7.2, JP1.2 (B), JP5.2 (B), Q1.3 (S), Q2.3 (S), R7.1, U3.3 (GND)
- new net: C11.1, U2.3 (VAUX)
- new net: J_USB_C1.A5 (CC1), R_CC1.1
- new net: R4.2, U1.1 (PS/SYNC), U1.14 (EN)
- new net: L1.2, U1.11 (L1)
- new net: R3.2, U1.2 (PG)
- new net: C1.1, U1.3 (VAUX)
- new net: R1.2, R2.1, U1.5 (FB)
- new net: L1.1, U1.9 (L2)
- new net: J_USB_C1.B5 (CC2), R_CC2.1
- new net: C7.1, R6.2
- new net: R7.2, SW1.3 (C)
- new net: Q1.2 (G), R6.1, SW1.2 (B)
- new net: JP6.2 (B), SW2.3 (C)
- new net: R_D+1.1, U_ESP32.14 (USB_D+)
- new net: R5.2, U2.1 (PS/SYNC), U2.14 (EN)
- new net: R_D-1.1, U_ESP32.13 (USB_D-)
- new net: L2.2, U2.11 (L1)
- new net: R10.2, U2.2 (PG)
- new net: R12.2, R9.1, U2.5 (FB)
- new net: L2.1, U2.9 (L2)
- new net: R12.1, R8.2
- new net: J_SD_Card1.1 (DAT2), R_SD_CARD2.2
- new net: R_ESP32_3.2, U_ESP32.15 (IO3)
- new net: JP_ESP32_9.2 (B), R_ESP32_46.2, U_ESP32.16 (IO46)
- new net: JP_ESP32_2.2 (B), R_ESP32_4.2, U_ESP32.27 (IO0)
- new net: R11.1, R9.2
- new net: J_SD_Card1.8 (DAT1), R_SD_CARD1.2
- new net +3V3: C_ESP32.1, J_Provide1.2 (Pin_2), J_Receive1.2 (Pin_2), J_SD_Card1.4 (VDD), R_ESP32_3.1, R_ESP32_4.1, R_ESP32_46.1, R_MISO1.1, R_MOSI1.1, R_SCL1.1, R_SDA1.1, R_SD_CARD1.1, R_SD_CARD2.1, R_SD_CARD_CS1.1, R_nReset1.1, U_ESP32.2 (3V3)
- new net +5V: J_Provide1.3 (Pin_3), J_Receive1.3 (Pin_3)
- new net 3V3: C16.1, C17.1, C4.1, C5.1, R1.1, R3.1, U1.7 (VOUT), U1.8 (VOUT)
- new net 5V: C12.1, C13.1, C14.1, C15.1, R10.1, R8.1, U2.7 (VOUT), U2.8 (VOUT)
- new net AD1: J_Provide1.12 (Pin_12), U_ESP32.39 (IO1)
- new net AD2: J_Provide1.13 (Pin_13), U_ESP32.38 (IO2)
- new net AD4: J_Provide2.1 (Pin_1), U_ESP32.4 (IO4)
- new net AD5: J_Provide2.2 (Pin_2), U_ESP32.5 (IO5)
- new net AD6: J_Provide2.3 (Pin_3), U_ESP32.6 (IO6)
- new net AD7: J_Provide2.4 (Pin_4), U_ESP32.7 (IO7)
- new net BATTERY_OK: Q2.2 (G), U3.1 (~{RESET})
- new net BATTERY_TO_SWITCH: JP3.2 (B), SW2.1 (A)
- new net CS_SD_Card: J_SD_Card1.2 (DAT3/CD), R_SD_CARD_CS1.2, U_ESP32.18 (IO10)
- new net Config1: J_Config1.1 (Pin_1), U_ESP32.34 (IO41)
- new net Config2: J_Config1.3 (Pin_3), U_ESP32.35 (IO42)
- new net Config3: J_Config1.5 (Pin_5), U_ESP32.26 (IO45)
- new net D14: J_Provide2.5 (Pin_5), U_ESP32.22 (IO14)
- new net D15: J_Provide2.6 (Pin_6), U_ESP32.8 (IO15)
- new net D16: J_Provide2.7 (Pin_7), U_ESP32.9 (IO16)
- new net D17: J_Provide2.8 (Pin_8), U_ESP32.10 (IO17)
- new net D18: J_Provide2.9 (Pin_9), U_ESP32.11 (IO18)
- new net D38: J_Provide2.10 (Pin_10), U_ESP32.31 (IO38)
- new net D39: J_Provide2.11 (Pin_11), U_ESP32.32 (IO39)
- new net D40: J_Provide2.12 (Pin_12), U_ESP32.33 (IO40)
- new net GNDREF: C1.2, C10.2, C11.2, C12.2, C13.2, C14.2, C15.2, C16.2, C17.2, C2.2, C3.2, C4.2, C5.2, C6.2, C8.2, C9.2, C_ESP32.2, JP1.1 (A), JP5.1 (A), JP_ESP32_2.1 (A), JP_ESP32_9.1 (A), J_Config1.2 (Pin_2), J_Config1.4 (Pin_4), J_Config1.6 (Pin_6), J_Program1.1 (Pin_1), J_Provide1.1 (Pin_1), J_Provide2.13 (Pin_13), J_Receive1.1 (Pin_1), J_SD_Card1.6 (VSS), J_Share1.2 (Pin_2), J_USB_C1.A1 (GND), J_USB_C1.A12 (GND), J_USB_C1.B1 (GND), J_USB_C1.B12 (GND), Q1.1 (D), Q2.1 (D), R11.2, R2.2, R_CC1.2, R_CC2.2, SW_nReset1.2, U1.10 (PGND), U1.4 (GND), U1.6 (FB2), U2.10 (PGND), U2.4 (GND), U2.6 (FB2), U_ESP32.1 (GND), U_ESP32.40 (GND), U_ESP32.41 (GND)
- new net I2C_SCL: J_Provide1.8 (Pin_8), J_Receive1.4 (Pin_4), R_SCL1.2, U_ESP32.17 (IO9)
- new net I2C_SDA: J_Provide1.7 (Pin_7), J_Receive1.5 (Pin_5), R_SDA1.2, U_ESP32.12 (IO8)
- new net Low_Battery: J_Receive1.6 (Pin_6), U_ESP32.25 (IO48)
- new net SPI_MISO: J_Provide1.9 (Pin_9), J_SD_Card1.7 (DAT0), R_MISO1.2, U_ESP32.21 (IO13)
- new net SPI_MOSI: J_Provide1.10 (Pin_10), J_SD_Card1.3 (CMD), R_MOSI1.2, U_ESP32.19 (IO11)
- new net SPI_SCK: J_Provide1.11 (Pin_11), J_SD_Card1.5 (CLK), U_ESP32.20 (IO12)
- new net UART_RX: J_Provide1.5 (Pin_5), U_ESP32.37 (TXD0)
- new net UART_TX: J_Provide1.6 (Pin_6), U_ESP32.36 (RXD0)
- new net USB_D+: J_Program1.4 (Pin_4), J_USB_C1.A6 (D+), J_USB_C1.B6 (D+), R_D+1.2
- new net USB_D-: J_Program1.3 (Pin_3), J_USB_C1.A7 (D-), J_USB_C1.B7 (D-), R_D-1.2
- new net USB_V: J_Program1.2 (Pin_2), J_USB_C1.A4 (VBUS), J_USB_C1.A9 (VBUS), J_USB_C1.B4 (VBUS), J_USB_C1.B9 (VBUS)
- new net V+: JP3.1 (A), JP4.1 (A)
- new net V_BATTERY: C10.1, C2.1, C3.1, C6.1, C8.1, C9.1, JP4.2 (B), R4.1, R5.1, SW1.1 (A), SW2.2 (B), U1.12 (VIN), U1.13 (VIN), U2.12 (VIN), U2.13 (VIN), U3.4 (VDD)
- new net nEnable_Share: J_Share1.1 (Pin_1), U_ESP32.24 (IO47)
- new net nReset: J_Provide1.4 (Pin_4), R_nReset1.2, SW_nReset1.1, U_ESP32.3 (EN)
- no-connect marks 0 -> 13
Other:
- note added: "3V3 and 5V voltage regulation circuits. Capacitor and resistor values haven't been chosen yet."
- note added: "3V3 voltage regulator"
- note added: "5.6V if fully charged 4.6V is nominal 4.0V is low battery 3.4V is battery critically low"
- note added: "5V voltage regulator"
- note added: "Device can operate in power save mode if PS/SYNC is set to high."
- note added: "Disables power to the sensor module when the battery is critically low."
- note added: "Switch circuit"
- note added: "This is Hannah's spot"
- note removed: "NETWORK SUBSYSTEM"

Commit message: Integrated Hannah's PCB onto the main circuit. Now I have to do a force push.
Parts:
- added J1: Conn_01x14_Pin, Connector_PinHeader_2.54mm:PinHeader_1x14_P2.54mm_Vertical, symbol Connector:Conn_01x14_Pin
- added J2, J6, J7: Conn_01x12_Pin, Connector_PinHeader_2.54mm:PinHeader_1x12_P2.54mm_Vertical, symbol Connector:Conn_01x12_Pin
- added J3, J5: Conn_01x08_Pin, Connector_PinHeader_2.54mm:PinHeader_1x08_P2.54mm_Vertical, symbol Connector:Conn_01x08_Pin
- added J4: Conn_01x14_Pin, Connector_PinSocket_2.54mm:PinSocket_1x14_P2.54mm_Vertical, symbol Connector:Conn_01x14_Pin
- added U4: ESP32-S3-WROOM-1U-N8, ESP32-WROOM-32UE_N4:ESP32-S3-WROOM-1U_No_holes, symbol ESP32-S3-WROOM-1U.pretty:ESP32-S3-WROOM-1U
- added U5: LORA-CC68-433MHz-TCXO, LORA-CC68-433MHz-TCXO:LORA-CC68-433MHz-TCXO, symbol LORA-CC68-433MHz-TCXO:LoRa-CC68_433MHz-TCXO
- added U6: ATGM332D-5N71, ATGM332D-5NR32:ATGM332D-5NR32, symbol ATGM332D-5NR32:ATGM332D-5NR32
Connections:
- net GND: now also J1.1 (Pin_1), J3.1 (Pin_1), J3.8 (Pin_8), J4.14 (Pin_14), J5.7 (Pin_7), J6.1 (Pin_1), J6.12 (Pin_12), J7.1 (Pin_1), U4.1 (GND), U4.40 (GND), U4.41 (GND), U5.1 (GND), U5.10 (GND), U5.8 (GND), U6.12 (GND), U6.13 (GND), U6.24 (GND)
- new net: J5.6 (Pin_6), U5.11 (DIO3)
- new net: J5.5 (Pin_5), U5.12 (NC)
- new net: J5.4 (Pin_4), U5.13 (VCC)
- new net: J5.3 (Pin_3), U5.14 (NC)
- new net: J5.2 (Pin_2), U5.15 (DIO1)
- new net: J5.1 (Pin_1), U5.16 (BUSY)
- new net: J3.2 (Pin_2), U5.2 (MISO)
- new net: J3.3 (Pin_3), U5.3 (MOSI)
- new net: J3.4 (Pin_4), U5.4 (SCK)
- new net: J3.5 (Pin_5), U5.5 (NSS)
- new net: J3.6 (Pin_6), U5.6 (NRESET)
- new net: J3.7 (Pin_7), U5.7 (NC)
- new net: J5.8 (Pin_8), U5.9 (ANT)
- new net: J6.10 (Pin_10), U6.22 (VBAT)
- new net: J6.11 (Pin_11), U6.23 (VCC)
- new net: J6.2 (Pin_2), U6.14 (NC)
- new net: J6.3 (Pin_3), U6.15 (NC)
- new net: J6.4 (Pin_4), U6.16 (TXD2)
- new net: J6.5 (Pin_5), U6.17 (RXD2)
- new net: J6.6 (Pin_6), U6.18 (SDA)
- new net: J6.7 (Pin_7), U6.19 (SCL)
- new net: J6.8 (Pin_8), U6.20 (TXD1)
- new net: J6.9 (Pin_9), U6.21 (RXD1)
- new net: J7.12 (Pin_12), U6.1 (NC)
- new net: J7.3 (Pin_3), U6.10 (GND)
- new net: J7.2 (Pin_2), U6.11 (RF_IN)
- new net: J7.11 (Pin_11), U6.2 (Reserved)
- new net: J7.10 (Pin_10), U6.3 (1PPS)
- new net: J7.9 (Pin_9), U6.4 (Reserved)
- new net: J7.8 (Pin_8), U6.5 (NC)
- new net: J7.7 (Pin_7), U6.6 (NC)
- new net: J7.6 (Pin_6), U6.7 (NC)
- new net: J7.5 (Pin_5), U6.8 (nRESET)
- new net: J7.4 (Pin_4), U6.9 (VCC_RF)
- new net 10: J1.10 (Pin_10), U4.10 (IO17)
- new net 11: J1.11 (Pin_11), U4.11 (IO18)
- new net 12: J1.12 (Pin_12), U4.12 (IO8)
- new net 13: J1.13 (Pin_13), U4.13 (IO19)
- new net 14: J1.14 (Pin_14), U4.14 (IO20)
- new net 15: J2.1 (Pin_1), U4.15 (IO3)
- new net 16: J2.2 (Pin_2), U4.16 (IO46)
- new net 17: J2.3 (Pin_3), U4.17 (IO9)
- new net 18: J2.4 (Pin_4), U4.18 (IO10)
- new net 19: J2.5 (Pin_5), U4.19 (IO11)
- new net 2: J1.2 (Pin_2), U4.2 (3V3)
- new net 20: J2.6 (Pin_6), U4.20 (IO12)
- new net 21: J2.7 (Pin_7), U4.21 (IO13)
- new net 22: J2.8 (Pin_8), U4.22 (IO14)
- new net 23: J2.9 (Pin_9), U4.23 (IO21)
- new net 24: J2.10 (Pin_10), U4.24 (IO47)
- new net 25: J2.11 (Pin_11), U4.25 (IO48)
- new net 26: J2.12 (Pin_12), U4.26 (IO45)
- new net 27: J4.1 (Pin_1), U4.27 (IO0)
- new net 28: J4.2 (Pin_2), U4.28 (IO35)
- new net 29: J4.3 (Pin_3), U4.29 (IO36)
- new net 3: J1.3 (Pin_3), U4.3 (EN)
- new net 30: J4.4 (Pin_4), U4.30 (IO37)
- new net 31: J4.5 (Pin_5), U4.31 (IO38)
- new net 32: J4.6 (Pin_6), U4.32 (IO39)
- new net 33: J4.7 (Pin_7), U4.33 (IO40)
- new net 34: J4.8 (Pin_8), U4.34 (IO41)
- new net 35: J4.9 (Pin_9), U4.35 (IO42)
- new net 36: J4.10 (Pin_10), U4.36 (RXD0)
- new net 37: J4.11 (Pin_11), U4.37 (TXD0)
- new net 38: J4.12 (Pin_12), U4.38 (IO2)
- new net 39: J4.13 (Pin_13), U4.39 (IO1)
- new net 4: J1.4 (Pin_4), U4.4 (IO4)
- new net 5: J1.5 (Pin_5), U4.5 (IO5)
- new net 6: J1.6 (Pin_6), U4.6 (IO6)
- new net 7: J1.7 (Pin_7), U4.7 (IO7)
- new net 8: J1.8 (Pin_8), U4.8 (IO15)
- new net 9: J1.9 (Pin_9), U4.9 (IO16)
Other:
- note added: "NETWORK SUBSYSTEM"
- moved on the sheet: Q2
